File: hackpadbludprint.kicad_sch (KiCad schematic)
At the start: 0 parts

Commit message: Stretch 1
- Schematic
- PCB
Parts:
- added SW1, SW2, SW3: SW_Push, Button_Switch_Keyboard:SW_Cherry_MX_1.00u_PCB, symbol Switch:SW_Push
- added U1: MOUDLE-SEEEDUINO-XIAO, HC Care Package footprints:XIAO-Generic-Hybrid-14P-2.54-21X17.8MM, symbol XIAO_RP2040:MOUDLE-SEEEDUINO-XIAO
Connections:
- new net: SW2.1, U1.10 (PA5_A9_D9_MISO)
- new net: SW1.1, U1.11 (PA6_A10_D10_MOSI)
- new net: SW3.1, U1.9 (PA7_A8_D8_SCK)
- new net GND: SW1.2, SW2.2, SW3.2, U1.13 (GND)
