File: pcb/hackpadbludprint.kicad_sch (KiCad schematic)
At the start: 4 parts, among them SW1 SW_Push, SW2 SW_Push, SW3 SW_Push, U1 MOUDLE-SEEEDUINO-XIAO

Commit message: Reorganizing files
Parts:
- added D2: SK6812MINI-E, LED_SMD:LED_SK6812MINI-E_3.2x2.8mm_P1.5mm_ReverseMount, symbol LED:SK6812MINI-E
- added SW4: SW_Push, Button_Switch_Keyboard:SW_Cherry_MX_1.00u_PCB, symbol Switch:SW_Push
Connections:
- net GND: now also D2.1 (VSS), SW4.2
- net at U1.5 (PA8_A4_D4_SDA): now also D2.2 (DIN)
- net at U1.8 (PB09_A7_D7_RX): now also SW4.1
- new net +5V: D2.3 (VDD)
Other:
- moved on the sheet: SW3

Commit message: STRETCH 3!!!!
- board looking nice
- Tysm jame
Parts:
- added D2, D3, D4: SK6812MINI-E, LED_SMD:LED_SK6812MINI-E_3.2x2.8mm_P1.5mm_ReverseMount, symbol LED:SK6812MINI-E
- added SW5: RotaryEncoder_Switch, Rotary_Encoder:RotaryEncoder_Alps_EC11E-Switch_Vertical_H20mm, symbol Device:RotaryEncoder_Switch
- added U2: ER_OLEDM0.91_1x-I2C, Display:ER_OLEDM0.91_1x-I2C, symbol Display_Graphic:ER_OLEDM0.91_1x-I2C
- renumbered D2 to D1
Connections:
- net +5V: now also U1.14 (5V), D2.3 (VDD), D3.3 (VDD), D4.3 (VDD), U2.2 (VCC)
- net GND: now also D2.1 (VSS), D3.1 (VSS), D4.1 (VSS), SW5.C, SW5.S2, U2.1 (GND)
- net at D1.2 (DIN): now also U1.7 (PB08_A6_D6_TX); no longer U1.5 (PA8_A4_D4_SDA)
- net at D1.4 (DOUT): now also D2.2 (DIN)
- net at U1.1 (PA02_A0_D0): now also SW5.B
- net at U1.2 (PA4_A1_D1): now also SW5.A
- net at U1.3 (PA10_A2_D2): now also SW5.S1
- net at U1.6 (PA9_A5_D5_SCL): now also U2.3 (SCL)
- new net: U1.5 (PA8_A4_D4_SDA), U2.4 (SDA)
- new net: D3.4 (DOUT), D4.2 (DIN)
- new net: D2.4 (DOUT), D3.2 (DIN)
Other:
- title: (none) -> Henry Wau's Bludpad
- moved on the sheet: D1
