File: pcb/hackpadbludprint.kicad_pcb (KiCad board)
At the start: 2 copper layers, 38.7 x 97.8 mm, 12 parts, among them SW1 SW_Push, SW2 SW_Push, SW3 SW_Push, SW4 SW_Push, SW5 RotaryEncoder_Switch, U1 MOUDLE-SEEEDUINO-XIAO, U2 ER_OLEDM0.91_1x-I2C

Commit message: TRYING TO FIX FIRMWARE
- Changed pcb silkscreen
- Moved readmes
Parts:
- removed the G*** at (166.5, 126.0)
- added G***: LOGO, projftprints:dragonbridge, F.Cu at (167.0, 127.0)
